File: Schematic/_autosave-edesign344-schematic-27163296.kicad_sch (KiCad schematic)
At the start: 63 parts, among them Q1 2N3906, Q2 2N3904, SW1 SW_Rotary_4x3, SW2 SW_Rotary_4x3, U1 NE555P, U2 TL081, U3 TL081, U4 TL081, U5 TL081, U6 TL081, U7 TL081, U8 TL081, U9 TL081

Commit message: backup
Connections:
- net Bridge-C1-A renamed Sine-C1-B
- net Sine-C1-B: no longer SW2.B
- net Bridge-C2-A renamed Sine-C2-B
- net Sine-C2-B: no longer SW2.A
- new net Sine-C1-A: SW2.B
- new net Sine-C2-A: SW2.A
Changed lines of the file:
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@@
 		)
 	)
-	(global_label "Bridge-C1-A"
+	(global_label "Sine-C1-A"
 		(shape input)
 		(at 246.38 71.12 0)
@@
 		)
 		(property "Intersheetrefs" "${INTERSHEET_REFS}"
-			(at 262.1257 71.12 0)
-			(effects
-				(font
-					(size 1.27 1.27)
-				)
-				(justify left)
-				(hide yes)
-			)
-		)
-	)
-	(global_label "Bridge-C2-A"
+			(at 260.13 71.12 0)
+			(effects
+				(font
+					(size 1.27 1.27)
+				)
+				(justify left)
+				(hide yes)
+			)
+		)
+	)
+	(global_label "Sine-C2-B"
 		(shape input)
 		(at 265.43 118.11 180)
@@
 		)
 		(property "Intersheetrefs" "${INTERSHEET_REFS}"
-			(at 249.6843 118.11 0)
+			(at 251.4986 118.11 0)
 			(effects
 				(font
@@
 		)
 	)
-	(global_label "Bridge-C1-A"
+	(global_label "Sine-C1-B"
 		(shape input)
 		(at 247.65 118.11 180)
@@
 		)
 		(property "Intersheetrefs" "${INTERSHEET_REFS}"
-			(at 231.9043 118.11 0)
+			(at 233.7186 118.11 0)
 			(effects
 				(font
@@
 		)
 	)
-	(global_label "Bridge-C2-A"
+	(global_label "Sine-C2-A"
 		(shape input)
 		(at 254 74.93 0)
@@
 		)
 		(property "Intersheetrefs" "${INTERSHEET_REFS}"
-			(at 269.7457 74.93 0)
-			(effects
-				(font
+			(at 267.75 74.93 0)
+			(effects
+				(font

Commit message: backup
Parts:
- removed C8, C9: C, symbol Device:C
Connections:
- net Sine-C1-A: now also R11.1, R12.1, U6.2 (-), U6.6
- net Sine-C1-B: now also R12.2, R16.1, U5.3 (+)
- net Sine-C2-A: now also R16.2
- net Sine-C2-B: now also D5.1 (K), D6.2 (A), R14.2, U5.6
Other:
- moved on the sheet: D5, D6, R12, R14, R16
