File: Schematic/edesign344-schematic-27163296.kicad_sch (KiCad schematic)
At the start: 62 parts, among them Q1 2N3906, Q2 2N3904, SW1 SW_Rotary_4x3, SW2 SW_Rotary_4x3, U1 NE555P, U2 TL081, U3 TL081, U4 TL081, U5 TL081, U6 TL081, U7 TL081, U8 TL081, U9 TL081

Commit message: backup
Parts:
- added R25: 20k, symbol Device:R
- R22, R23: value 220 -> 68k
- RV3: value R_Potentiometer -> 100k
Connections:
- net at R18.2, U7.6, U8.3 (-): now also R25.1; no longer U8.6
- net 15V-VGND: now reaches U7.2 (+)
- new net: R25.2, U8.6
Other:
- note added: "Signal selection, gain and offset op-amp circuits"
Changed lines of the file:
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@@
 		)
 	)
-	(text "SINE WAVE - Wien bridge"
+	(text "Signal selection, gain and offset op-amp circuits"
 		(exclude_from_sim no)
-		(at 30.48 17.78 0)
+		(at 41.91 17.526 0)
 		(effects
 			(font
@@
 	(wire
 		(pts
-			(xy 80.01 50.8) (xy 80.01 48.26)
+			(xy 81.28 52.07) (xy 81.28 48.26)
 		)
 		(stroke
@@
 	(wire
 		(pts
-			(xy 116.84 34.29) (xy 135.89 34.29)
+			(xy 116.84 34.29) (xy 123.19 34.29)
 		)
 		(stroke
@@
 	(wire
 		(pts
+			(xy 130.81 34.29) (xy 135.89 34.29)
+		)
+		(stroke
+			(width 0)
+			(type default)
+		)
+	)
+	(wire
+		(pts
 			(xy 48.26 45.72) (xy 50.8 45.72)
 		)
@@
 	(wire
 		(pts
-			(xy 80.01 48.26) (xy 83.82 48.26)
+			(xy 81.28 48.26) (xy 83.82 48.26)
 		)
 		(stroke
@@
 		)
 	)
+	(global_label "15V-VGND"
+		(shape input)
+		(at 81.28 52.07 270)
+		(fields_autoplaced yes)
+		(effects
+			(font
+				(size 1.27 1.27)
+			)
+			(justify right)
+		)
+		(property "Intersheetrefs" "${INTERSHEET_REFS}"
+			(at 81.28 65.0943 90)
+			(effects
+				(font
+					(size 1.27 1.27)
+				)
+				(justify right)
+				(hide yes)
+			)
+		)
+	)
 	(global_label "Sqr-Tri-PWR"
 		(shape input)
@@
 		(on_board yes)
 		(dnp no)
-		(fields_autoplaced yes)
 		(property "Reference" "SW1"
-			(at 62.865 17.78 0)
+			(at 63.5 21.336 0)
 			(effects
 				(font
@@
 		)
 		(property "Value" "SW_Rotary_4x3"
-			(at 62.865 20.32 0)
+			(at 62.992 60.452 0)
 			(effects
 				(font
@@
 			)
 		)
-		(property "Value" "220"
+		(property "Value" "68k"
 			(at 119.38 61.976 90)
 			(effects
@@
 	)
 	(symbol
+		(lib_id "Device:R")
+		(at 127 34.29 90)
+		(unit 1)
+		(exclude_from_sim no)
+		(in_bom yes)
+		(on_board yes)
+		(dnp no)
+		(property "Reference" "R25"
+			(at 127 32.004 90)
+			(effects
+				(font
+					(size 1.27 1.27)
+				)
+			)
+		)
+		(property "Value" "20k"
+			(at 127 36.576 90)
+			(effects
+				(font
+					(size 1.27 1.27)
+				)
+			)
+		)
+		(property "Footprint" ""
+			(at 127 36.068 90)
+			(effects
+				(font
+					(size 1.27 1.27)
+				)
+				(hide yes)
+			)
+		)
+		(property "Datasheet" "~"
+			(at 127 34.29 0)
+			(effects
+				(font
+					(size 1.27 1.27)
+				)
+				(hide yes)
+			)
+		)
+		(property "Description" "Resistor"
+			(at 127 34.29 0)
+			(effects
+				(font
+					(size 1.27 1.27)
+				)
+				(hide yes)
+			)
+		)
+		(pin "2"
+		)
+		(pin "1"
+		)
+		(instances
+			(project "edesign344-schematic-27163296"
+				(path "/231675ab-32c5-49c0-9bd3-8a612300c001"
+					(reference "R25")
+					(unit 1)
+				)
+			)
+		)
+	)
+	(symbol
 		(lib_id "power:GND")
 		(at 44.45 147.32 0)
@@
 			)
 		)
-		(property "Value" "220"
+		(property "Value" "68k"
 			(at 104.14 61.976 90)
 			(effects
@@
 		)
 		(property "Value" "GND"
-			(at 84.328 55.626 0)
+			(at 91.948 53.594 0)
 			(effects
 				(font
@@
 			)
 		)
-		(property "Value" "R_Potentiometer"
-			(at 111.76 64.262 90)
+		(property "Value" "100k"
+			(at 112.014 62.23 90)
 			(effects
 				(font

Commit message: backup
Parts:
- removed C8, C9: C, symbol Device:C
Connections:
- net Sine-C2-B: now reaches D5.1 (K), D6.2 (A), R14.2, U5.6
- net Sine-C2-B: now also C13.2, C14.2, C15.2
- net Sine-C1-A: now reaches R11.1, R12.1, U6.2 (-), U6.6
- net Sine-C1-A: now also SW2.B
- net Sine-C1-B: now reaches R12.2, R16.1, U5.3 (+)
- net Sine-C1-B: now also C1.2, C11.2, C12.2
- net Sine-C2-A: now reaches R16.2
- net Sine-C2-A: now also SW2.A
- removed net Bridge-C1-A: C1.2, C11.2, C12.2, SW2.B
- removed net Bridge-C2-A: C13.2, C14.2, C15.2, SW2.A
Other:
- moved on the sheet: D5, D6, R12, R14, R16
